File: TFG/TFG.kicad_sch (KiCad schematic)
At the start: 36 parts, among them IC1 MC74VHC1GT14DBVT1G, IC2 AMS1117-5.0, IC3 AMS1117-5.0, J1 Jack-DC, J2 CON-SMA-EDGE-SRP, J3 CON-SMA-EDGE-SRP, Q1 BFP420

Commit message: BOM Uploaded but SRD and Schottky diodes are pending
Parts:
- BFR35AP: renamed from BFG135A1; footprint Package_TO_SOT_SMD:SOT-223 -> Package_TO_SOT_SMD:SOT-23
Changed lines of the file:
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@@
 		(dnp no)
 		(fields_autoplaced yes)
-		(property "Reference" "BFG135A1"
+		(property "Reference" "BFR35AP"
 			(at 165.1 102.8699 0)
 			(effects
@@
 			)
 		)
-		(property "Footprint" "Package_TO_SOT_SMD:SOT-223"
+		(property "Footprint" "Package_TO_SOT_SMD:SOT-23"
 			(at 165.1 101.6 0)
 			(effects
@@
 			(project "TFG"
 				(path "/f38180f0-5f14-4552-a9c5-56b7688c9594"
-					(reference "BFG135A1")
+					(reference "BFR35AP")
 					(unit 1)
 				)

Commit message: Power islands and vias placement, only we re missing diodes models
Parts:
- IC2, IC3: value AMS1117-5.0 -> TS1117BCW50 RPG
Changed lines of the file:
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@@
 			)
 		)
-		(property "Value" "AMS1117-5.0"
+		(property "Value" "TS1117BCW50 RPG"
 			(at 50.8 157.48 0)
 			(effects
@@
 			)
 		)
-		(property "Value" "AMS1117-5.0"
+		(property "Value" "TS1117BCW50 RPG"
 			(at 152.4 24.13 0)
 			(effects

Commit message: Updated Schottky and SRD diodes in PCB and BOM, everything is ready to check, only DRC is missing
Parts:
- D1: renamed from D3; value D_Schottky_BAT15 -> SMS3923-079LF; footprint Diode_SMD:D_SOD-323 -> SMS3923-079LF:SODFL1608X70N
- D2: renamed from D1; value D_Schottky_BAT15 -> SMS3923-079LF; footprint Diode_SMD:D_SOD-323 -> SMS3923-079LF:SODFL1608X70N
- D3: renamed from D2; value SRD_ASRD808D -> SRD_MA144769-287T; footprint Diode_SMD:D_SOD-323 -> MA144769287T; symbol Device:D -> MA144769-287T:MA144769-287T; Height (none) -> 1.22; Manufacturer_Name (none) -> MACOM; Manufacturer_Part_Number (none) -> MA144769-287T; Mouser Part Number (none) -> 937-MA144769-287T; Mouser Price/Stock (none) -> https://www.mouser.co.uk/ProductDetail/MACOM/MA144769-287T?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
- IC1: value MC74VHC1GT14DBVT1G -> MC74VHC1GT04DFT2G; footprint SOT95P275X110-5N -> MC74VHC1GT04DFT2G:SOT65P210X110-5N
- renumbered BFR35AP to BFR35AP1, C12 to C1, C9 to C10, C6 to C11, C11 to C12, C3 to C13, C13 to C14, C14 to C15, C4 to C16, C7 to C2, C8 to C3, C15 to C4, C16 to C5, C2 to C6, C1 to C7, C5 to C8, C10 to C9, R4 to R3, R3 to R4, R6 to R5, R7 to R6, R8 to R7, R9 to R8
Connections:
- net GND: now also D3.3 (K); no longer D3.1 (K)
- net at C13.2, C16.1, D1.1 (K)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: now also D3.1 (A); no longer D3.2 (A)
Other:
- moved on the sheet: D1

Commit message: Final design for Ultrawideband pulse generator PCB - v1
Parts:
- J1: symbol Connector:Jack-DC -> Connector:Barrel_Jack_Switch
Connections:
- net GND: now also J1.3
